File: UV_light.kicad_pcb (KiCad board)
At the start: 2 copper layers, 91 x 69 mm, 101 parts, among them P1 SMD_CONN, P10 SMD_CONN, P2 SMD_CONN, P3 SMD_CONN, P4 SMD_CONN, P5 CONN_01X01, P6 CONN_01X01, P7 SMD_CONN, P8 SMD_CONN, P9 SMD_CONN

Commit message: Comleting version 2
Parts:
- removed C2: 2.2uF, Local:Capacitor_Panasonic_G13
- added R13: 1M, Resistors_SMD:R_1206, F.Cu at (158.0, 75.2)
- C1: value 2.2uF -> 1uF; footprint Local:Capacitor_17.5x10x15mm -> Local:Capacitor_film_26.5x10
- C3: value 330uF -> 47uF; footprint Capacitors_SMD:c_elec_8x10 -> Local:Capacitor_Panasonic_G13
- P5, P6: footprint Local:TESTPOINT_SMD -> Local:TESTPOINT_SMD_3MM
- R1, R2: value 50R -> 1k3; footprint Resistors_SMD:R_0603 -> Resistors_SMD:R_2512; moved to F.Cu
- R3: value 50R -> 1M; footprint Resistors_SMD:R_0603 -> Resistors_SMD:R_1206; moved to F.Cu
- R4, R5, R6: value 50R -> 330R; footprint Resistors_SMD:R_0603 -> Resistors_SMD:R_1206
- moved R1 69.6 mm to (122.1, 98.4), turned to 270 degrees
- moved R2 62.9 mm to (132.9, 98.4), turned to 270 degrees
- moved R3 46.2 mm to (140.4, 98.4), turned to 180 degrees
- moved F1 35.6 mm to (127.6, 108.4), turned to 90 degrees
- moved R5 19.4 mm to (182.5, 87.2)
- moved R4 13.9 mm to (182.6, 75.8)
- moved G*** 8.78 mm to (161.8, 92.2)
- moved C3 6.50 mm to (148.2, 75.2)
- moved P6 6.30 mm to (153.8, 87.0)
- moved G*** 4.70 mm to (122.5, 86.5)
- moved C1 4.07 mm to (122.8, 86.5), turned to 180 degrees
- moved P5 3.80 mm to (145.5, 87.0)
- moved D1 3.52 mm to (129.4, 74.0)
- moved R6 2.70 mm to (183.0, 109.2)
- moved G*** 2.22 mm to (110.0, 75.8)
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Connections:
- C1 pad 2: /LIVE -> Net-(C1-Pad2)
- D1 pad 2: Net-(D1-Pad2) -> /NEUTRAL
- D10 pad 2: VCC -> Net-(D10-Pad2)
- D11 pad 1: Net-(D11-Pad1) -> Net-(D10-Pad2)
- D11 pad 2: Net-(D10-Pad1) -> Net-(D11-Pad2)
- D12 pad 1: Net-(D12-Pad1) -> Net-(D11-Pad2)
- D12 pad 2: Net-(D11-Pad1) -> Net-(D12-Pad2)
- D13 pad 1: Net-(D13-Pad1) -> Net-(D12-Pad2)
- D13 pad 2: Net-(D12-Pad1) -> Net-(D13-Pad2)
- D14 pad 1: Net-(D14-Pad1) -> Net-(D13-Pad2)
- D14 pad 2: Net-(D13-Pad1) -> Net-(D14-Pad2)
- D15 pad 1: Net-(D15-Pad1) -> Net-(D14-Pad2)
- D15 pad 2: Net-(D14-Pad1) -> Net-(D15-Pad2)
- D16 pad 1: Net-(D16-Pad1) -> Net-(D15-Pad2)
- D16 pad 2: Net-(D15-Pad1) -> Net-(D16-Pad2)
- D17 pad 1: Net-(D17-Pad1) -> Net-(D16-Pad2)
- D17 pad 2: Net-(D16-Pad1) -> Net-(D17-Pad2)
- D18 pad 2: VCC -> Net-(D18-Pad2)
- D2 pad 2: VCC -> Net-(D10-Pad1)
- D25 pad 1: Net-(D25-Pad1) -> GND
- D26 pad 1: Net-(D26-Pad1) -> Net-(D18-Pad2)
- D26 pad 2: VCC -> Net-(D26-Pad2)
- D27 pad 1: Net-(D27-Pad1) -> Net-(D26-Pad2)
- D27 pad 2: Net-(D26-Pad1) -> Net-(D27-Pad2)
- D28 pad 1: Net-(D28-Pad1) -> Net-(D27-Pad2)
- D28 pad 2: Net-(D27-Pad1) -> Net-(D28-Pad2)
- D29 pad 1: Net-(D29-Pad1) -> Net-(D28-Pad2)
- D29 pad 2: Net-(D28-Pad1) -> Net-(D29-Pad2)
- D30 pad 1: Net-(D30-Pad1) -> Net-(D29-Pad2)
- D30 pad 2: Net-(D29-Pad1) -> Net-(D30-Pad2)
- D31 pad 1: Net-(D31-Pad1) -> Net-(D30-Pad2)
- D31 pad 2: Net-(D30-Pad1) -> Net-(D31-Pad2)
- D32 pad 1: Net-(D32-Pad1) -> Net-(D31-Pad2)
- D32 pad 2: Net-(D31-Pad1) -> Net-(D32-Pad2)
- D33 pad 1: Net-(D33-Pad1) -> Net-(D32-Pad2)
- D33 pad 2: Net-(D32-Pad1) -> Net-(D33-Pad2)
- D34 pad 2: VCC -> Net-(D34-Pad2)
- D41 pad 1: Net-(D41-Pad1) -> GND
- D42 pad 1: Net-(D42-Pad1) -> Net-(D34-Pad2)
- D42 pad 2: VCC -> Net-(D42-Pad2)
- D43 pad 1: Net-(D43-Pad1) -> Net-(D42-Pad2)
- D43 pad 2: Net-(D42-Pad1) -> Net-(D43-Pad2)
- D44 pad 1: Net-(D44-Pad1) -> Net-(D43-Pad2)
- D44 pad 2: Net-(D43-Pad1) -> Net-(D44-Pad2)
- D45 pad 1: Net-(D45-Pad1) -> Net-(D44-Pad2)
- D45 pad 2: Net-(D44-Pad1) -> Net-(D45-Pad2)
- D46 pad 1: Net-(D46-Pad1) -> Net-(D45-Pad2)
- D46 pad 2: Net-(D45-Pad1) -> Net-(D46-Pad2)
- D47 pad 1: Net-(D47-Pad1) -> Net-(D46-Pad2)
- D47 pad 2: Net-(D46-Pad1) -> Net-(D47-Pad2)
- D48 pad 1: Net-(D48-Pad1) -> Net-(D47-Pad2)
- D48 pad 2: Net-(D47-Pad1) -> Net-(D48-Pad2)
- D49 pad 1: Net-(D49-Pad1) -> Net-(D48-Pad2)
- D49 pad 2: Net-(D48-Pad1) -> Net-(D49-Pad2)
- D9 pad 1: Net-(D9-Pad1) -> GND
- F1 pad 1: /NEUTRAL -> /LIVE
- F1 pad 2: Net-(D1-Pad2) -> Net-(F1-Pad2)
- R1 pad 1: Net-(D17-Pad1) -> Net-(C1-Pad2)
- R1 pad 2: GND -> Net-(F1-Pad2)
- R2 pad 1: Net-(D9-Pad1) -> Net-(C1-Pad2)
- R2 pad 2: GND -> Net-(F1-Pad2)
- R3 pad 1: Net-(D25-Pad1) -> Net-(C1-Pad1)
- R3 pad 2: GND -> Net-(C1-Pad2)
- R4 pad 1: Net-(D33-Pad1) -> VCC
- R4 pad 2: GND -> Net-(D17-Pad2)
- R5 pad 1: Net-(D41-Pad1) -> VCC
- R5 pad 2: GND -> Net-(D33-Pad2)
- R6 pad 1: Net-(D49-Pad1) -> VCC
- R6 pad 2: GND -> Net-(D49-Pad2)
Routing:
- net VCC: track 122.7 -> 167.1 mm, vias 1 -> 3
- net Net-(C1-Pad2): track 0.00 -> 40.5 mm
- net Net-(F1-Pad2): track 0.00 -> 16.4 mm
- net Net-(D34-Pad2): track 0.00 -> 11.0 mm
- net Net-(D18-Pad2): track 0.00 -> 11.0 mm
- net Net-(C1-Pad1): track 23.2 -> 31.9 mm
- net Net-(D43-Pad2): track 0.00 -> 7.90 mm
- net Net-(D43-Pad1): track 7.90 -> 0.00 mm
- net Net-(D42-Pad2): track 0.00 -> 7.90 mm
- net Net-(D42-Pad1): track 7.90 -> 0.00 mm
- net Net-(D27-Pad2): track 0.00 -> 7.90 mm
- net Net-(D27-Pad1): track 7.90 -> 0.00 mm
- net Net-(D26-Pad2): track 0.00 -> 7.90 mm
- net Net-(D26-Pad1): track 7.90 -> 0.00 mm
- net Net-(D11-Pad2): track 0.00 -> 7.90 mm
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- added copper zone on F.Cu, net Net-(C1-Pad2)
- added copper zone on F.Cu, net Net-(F1-Pad2)
Other:
- net class 220V: clearance 1.5 -> 2; trace_width 1.5 -> 2; via_dia 1 -> 1.5; via_drill 0.6 -> 0.8
- net class Dist added: clearance 1.5, trace_width 1.5, via_dia 0.6, via_drill 0.4
